File: UselessBox V2.kicad_pcb (KiCad board)
At the start: 2 copper layers, 47.1 x 46.6 mm, 23 parts, among them J2 Conn_01x03, J3 Conn_01x02_Female, SW1 SW_SPDT, SW2 SW_SPDT, U1 L7805CV, U2 LM555CN_NOPB

Commit message: added github silkscreen to pcb
Other:
- board text added: "https://github.com/leistimo/UselessBox.git"
Changed lines of the file:
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@@
   (general
     (thickness 1.6)
-    (drawings 19)
+    (drawings 20)
     (tracks 139)
     (zones 0)
@@
     )
   )
+  (gr_text https://github.com/leistimo/UselessBox.git (at 147.828 123.317) (layer B.SilkS)
+    (effects (font (size 1 1) (thickness 0.15)) (justify mirror))
+  )
   (gr_text "Useless Box V2\nTimothy S Leishman 4/12/2022" (at 163.576 102.489) (layer B.SilkS)

Commit message: corrected SERVO pinout
Parts:
- removed G***: LOGO, Kicad:TSL Technologies logo 16mm x 11mm
- removed G***: LOGO, Kicad:TNT Logo 12.6mm x 7mm
Connections:
- J2 pad 1: /5Vout -> Net-(J2-Pad1)
- J2 pad 2: Net-(J2-Pad2) -> /5Vout
- U2 pad 3: Net-(J2-Pad2) -> Net-(J2-Pad1)
Routing:
- net Net-(J2-Pad1): track 0.00 -> 37.9 mm
- net Net-(J2-Pad2): track 34.8 -> 0.00 mm
- net /5Vout: track 125.6 -> 157.8 mm

Commit message: added logos
Parts:
- added G***: LOGO, Kicad:TNT Logo 12.6mm x 7mm, B.Cu at (157.9, 94.4)
- added G***: LOGO, Kicad:TSL Technologies logo 16mm x 11mm, B.Cu at (160.1, 107.2)
Other:
- board text added: "BRN"
- board text added: "ORG"
- board text added: "RED"
