File: UselessBox V2.sch (KiCad schematic (older format))
At the start: 21 parts, among them J2 Conn_01x03, J3 Conn_01x02_Female, SW1 SW_SPDT, SW2 SW_SPDT, U1 L7805CV, U2 LM555CN_NOPB

Commit message: stl file done for base and arm also revised PCB switch
Connections:
- net 5V renamed 5Vout
Changed lines of the file:
@@
 EESchema Schematic File Version 4
+LIBS:UselessBox V2-cache
 EELAYER 30 0
 EELAYER END
@@
 	7700 3250 7700 3150
 Wire Wire Line
-	6900 2850 7400 2850
-Wire Wire Line
 	7700 3050 7700 2850
 Wire Wire Line
@@
 	5300 4350 5050 4350
 $Comp
-L power:PWR_FLAG #FLG0105
-U 1 1 625D6FA7
-P 7400 2850
-F 0 "#FLG0105" H 7400 2925 50  0001 C CNN
-F 1 "PWR_FLAG" H 7400 3023 50  0000 C CNN
-F 2 "" H 7400 2850 50  0001 C CNN
-F 3 "~" H 7400 2850 50  0001 C CNN
-	1    7400 2850
-	1    0    0    -1
-$EndComp
-Connection ~ 7400 2850
-Wire Wire Line
-	7400 2850 7700 2850
-$Comp
 L Switch:SW_SPDT SW1
 U 1 1 625D785C
@@
 Text Label 5350 4350 0    50   ~ 0
 GND
-Text Label 5400 3250 0    50   ~ 0
-5V
 Text Label 6300 2850 0    50   ~ 0
 5Vout
@@
 Wire Wire Line
 	3050 3100 2950 3100
+Wire Wire Line
+	6900 2850 7700 2850
 $EndSCHEMATC
